File: Schematic/OPL3_VGM_Player/OPL3_VGM_Player.kicad_pcb (KiCad board)
At the start: 2 copper layers, 80 x 57.2 mm, 61 parts, among them J1 USB_OTG, J2 Conn_02x03_Odd_Even, J3 Micro_SD_Card, J4 Conn_01x04, J5 Audio-Jack-3, SW1 SW_Push_Dual, SW2 SW_Push_Dual, SW3 SW_Push_Dual, SW4 SW_Push_Dual, SW5 SW_Push_Dual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

Commit message: pcb 2024.0
Parts:
- removed J5: Audio-Jack-3, Boom Precision Elec PJ-307C:Boom Precision Elec PJ-307C
- added J6: USB_C_Receptacle_USB2.0_16P, Connector_USB:USB_C_Receptacle_HRO_TYPE-C-31-M-12, F.Cu at (181.6, 88.0)
- added R10: 5.1k, Resistor_SMD:R_0603_1608Metric_Pad0.98x0.95mm_HandSolder, F.Cu at (182.6, 95.5)
- added R11: 5.1k, Resistor_SMD:R_0603_1608Metric_Pad0.98x0.95mm_HandSolder, F.Cu at (180.7, 95.5)
- J1: value USB_OTG -> PJ-307; footprint Connectors:USB_Mini-B -> my:PJ-307
- J3: footprint customMicroSD:SOFNG_TF_15x15_PUSH_PUSH -> my:GCT-MEM2055-00-190-01-A
- L1: footprint Inductors_SMD:L_0603 -> Inductor_SMD:L_0603_1608Metric_Pad1.05x0.95mm_HandSolder
- Y1: footprint Crystals:Crystal_SMD_HC49-SD -> Crystal:Crystal_SMD_SeikoEpson_TSX3225-4Pin_3.2x2.5mm_HandSoldering
- moved J1 31.2 mm to (212.7, 87.3), turned to 0 degrees
- moved C5 9.22 mm to (178.0, 99.6), turned to 180 degrees
- moved L1 5.77 mm to (178.0, 97.7)
- moved C7 4.08 mm to (179.1, 104.4), turned to -45 degrees
- moved C8 3.26 mm to (174.1, 109.4), turned to 135 degrees
- moved Y1 2.70 mm to (176.6, 106.9)
- moved J3 2.70 mm to (166.2, 99.8)
- moved C4 2.66 mm to (178.0, 95.8)
- moved C12 1.23 mm to (168.3, 101.6), turned to 0 degrees
Connections:
- C7 pad 1: Net-(C7-Pad1) -> Net-(U2-PD0/RCC_OSC_IN)
- J3 pad 1: Net-(J3-Pad1) -> unconnected-(J3-DAT2-Pad1)
- J3 pad 8: Net-(J3-Pad8) -> unconnected-(J3-DAT1-Pad8)
- J3 pad 9: Net-(J3-Pad9) -> unconnected-(J3-SHIELD-Pad9)
- RV1 pad 2: Net-(J5-Pad3) -> Net-(J1-PadR)
- RV1 pad 5: Net-(J5-Pad2) -> Net-(J1-PadT)
- SW1 pad 2: Net-(SW1-Pad2) -> unconnected-(SW1-Pad2)
- SW1 pad 3: Net-(SW1-Pad3) -> unconnected-(SW1-Pad3)
- SW2 pad 2: Net-(SW2-Pad2) -> unconnected-(SW2-Pad2)
- SW2 pad 4: Net-(SW2-Pad4) -> unconnected-(SW2-Pad4)
- SW3 pad 2: Net-(SW3-Pad2) -> unconnected-(SW3-Pad2)
- SW3 pad 4: Net-(SW3-Pad4) -> unconnected-(SW3-Pad4)
- SW4 pad 2: Net-(SW4-Pad2) -> unconnected-(SW4-Pad2)
- SW4 pad 4: Net-(SW4-Pad4) -> unconnected-(SW4-Pad4)
- SW5 pad 2: Net-(SW5-Pad2) -> unconnected-(SW5-Pad2)
- SW5 pad 4: Net-(SW5-Pad4) -> unconnected-(SW5-Pad4)
- U2 pad 10: Net-(U2-Pad10) -> unconnected-(U2-ADC1_IN0/ADC2_IN0/SYS_WKUP/TIM2_CH1/TIM2_ETR/USART2_CTS/PA0-Pad10)
- U2 pad 12: Net-(U2-Pad12) -> unconnected-(U2-ADC1_IN2/ADC2_IN2/TIM2_CH3/USART2_TX/PA2-Pad12)
- U2 pad 13: Net-(U2-Pad13) -> unconnected-(U2-ADC1_IN3/ADC2_IN3/TIM2_CH4/USART2_RX/PA3-Pad13)
- U2 pad 32: Net-(U2-Pad32) -> unconnected-(U2-ADC1_EXTI11/ADC2_EXTI11/CAN_RX/TIM1_CH4/USART1_CTS/USB_DM/PA11-Pad32)
- U2 pad 33: Net-(U2-Pad33) -> unconnected-(U2-CAN_TX/TIM1_ETR/USART1_RTS/USB_DP/PA12-Pad33)
- U2 pad 4: Net-(U2-Pad4) -> unconnected-(U2-PC15/ADC1_EXTI15/ADC2_EXTI15/RCC_OSC32_OUT-Pad4)
- U2 pad 5: Net-(C7-Pad1) -> Net-(U2-PD0/RCC_OSC_IN)
- U3 pad 4: Net-(U3-Pad4) -> unconnected-(U3-RTS-Pad4)
- U3 pad 5: Net-(U3-Pad5) -> unconnected-(U3-CTS-Pad5)
- U3 pad 6: Net-(U3-Pad6) -> unconnected-(U3-TNOW-Pad6)
- U4 pad 2: Net-(U4-Pad2) -> unconnected-(U4-IRQ-Pad2)
- U4 pad 22: Net-(U4-Pad22) -> unconnected-(U4-DOCD-Pad22)
- U4 pad 9: Net-(U4-Pad9) -> unconnected-(U4-TEST-Pad9)
- U5 pad 15: Net-(U5-Pad15) -> unconnected-(U5-TST2-Pad15)
- U6 pad 11: Net-(U6-Pad11) -> GND
- Y1 pad 2: Net-(C7-Pad1) -> GND
Routing:
- net Net-(J1-PadT): track 0.00 -> 18.6 mm
- net Net-(J5-Pad2): track 16.1 -> 0.00 mm
- net D2: track 42.7 -> 30.5 mm
- net Net-(J1-PadR): track 0.00 -> 11.1 mm
- net GND: track 52.7 -> 63.8 mm, vias 81 -> 95
- net Net-(U2-PD0/RCC_OSC_IN): track 0.00 -> 9.50 mm
- net VCC: track 64.6 -> 74.0 mm
- net D-: track 11.0 -> 20.2 mm
- net Net-(J5-Pad3): track 8.58 -> 0.00 mm
- net Net-(C7-Pad1): track 7.94 -> 0.00 mm
- net Net-(U2-PD1/RCC_OSC_OUT): track 13.8 -> 6.58 mm
- net SD_MOSI: track 35.8 -> 30.3 mm
- net D+: track 12.1 -> 15.8 mm
- net SD_CS: track 28.2 -> 31.5 mm
- net Net-(J6-CC2): track 0.00 -> 2.88 mm
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Other:
- outline, holes or cut-outs redrawn
- net class 3.3 removed
- net class 5v removed
- net class Default removed
- rule pad_to_mask_clearance: 0.051 -> 0
- board text added: "Rev 2024.0 by Uzix"
- board text removed: "JLCJLCJLCJLC"
